Commit message: commit before reverting affordance to a service

File: ws_description/urdf/_d435.urdf.xacro (robot description, xacro)
@@ -9,5 +9,5 @@
   <xacro:macro name="sensor_d435" params="parent prefix *origin">
     <xacro:property name="M_PI" value="3.1415926535897931" />
-    <xacro:include filename="$(find rob10)/urdf/_d435.gazebo.xacro"/>
+    <xacro:include filename="$(find ws_description)/urdf/_d435.gazebo.xacro"/>
     <!-- The following values are approximate, and the camera node
      publishing TF values with actual calibrated camera extrinsic values -->
@@ -44,6 +44,6 @@
         <geometry>
           <!-- <box size="${d435_cam_width} ${d435_cam_height} ${d435_cam_depth}"/> -->
-	  <mesh filename="package://rob10/urdf/meshes/d435.dae" />
-          <!--<mesh filename="package://rob10/urdf/meshes/d435/d435.dae" />-->
+	  <mesh filename="package://ws_description/urdf/meshes/d435.dae" />
+          <!--<mesh filename="package://ws_description/urdf/meshes/d435/d435.dae" />-->
         </geometry>
         <material name="aluminum"/>
